Commit message: rover&drone

File: rehab_exo_description/urdf/rehab_exo.urdf (robot description, URDF)
Before this commit: robot rehab_exo, 11 links, 10 joints
Links:
- added link left_shank_ext, mass 0.600; collision box size=0.0400 0.0400 0.1400; visual box size=0.0380 0.0340 0.1400
- added link left_thigh_ext, mass 0.800; collision box size=0.1600 0.0400 0.0600; visual box size=0.1600 0.0380 0.0550
- added link right_shank_ext, mass 0.600; collision box size=0.0400 0.0400 0.1400; visual box size=0.0380 0.0340 0.1400
- added link right_thigh_ext, mass 0.800; collision box size=0.1600 0.0400 0.0600; visual box size=0.1600 0.0380 0.0550
- link left_thigh: geometry collision box size=0.4000 0.0600 0.0800; visual box size=0.4000 0.0500 0.0700
- link right_thigh: geometry collision box size=0.4000 0.0600 0.0800; visual box size=0.4000 0.0500 0.0700
Joints:
- removed joint base_to_seat
- added joint left_shank_ext_joint: type prismatic, parent left_shank, child left_shank_ext, origin xyz=0 0 -0.400 rpy=0 0 0, axis 0 0 -1, limit lower=0.0 upper=0.08 effort=300.0 velocity=0.03
- added joint left_thigh_ext_joint: type prismatic, parent left_thigh, child left_thigh_ext, origin xyz=0.400 0 0 rpy=0 0 0, axis 1 0 0, limit lower=0.0 upper=0.08 effort=300.0 velocity=0.03
- added joint right_shank_ext_joint: type prismatic, parent right_shank, child right_shank_ext, origin xyz=0 0 -0.400 rpy=0 0 0, axis 0 0 -1, limit lower=0.0 upper=0.08 effort=300.0 velocity=0.03
- added joint right_thigh_ext_joint: type prismatic, parent right_thigh, child right_thigh_ext, origin xyz=0.400 0 0 rpy=0 0 0, axis 1 0 0, limit lower=0.0 upper=0.08 effort=300.0 velocity=0.03
- added joint seat_lift_joint: type prismatic, parent base_link, child seat_link, origin xyz=0 0 0.485 rpy=0 0 0, axis 0 0 1, limit lower=0.0 upper=0.15 effort=500.0 velocity=0.05
- joint left_ankle_joint: origin xyz=0 0 -0.400 rpy=0 0 0 -> xyz=0 0 0 rpy=0 0 0; parent left_shank -> left_shank_ext
- joint left_knee_joint: origin xyz=0.400 0 0 rpy=0 0 0 -> xyz=0 0 0 rpy=0 0 0; parent left_thigh -> left_thigh_ext
- joint right_ankle_joint: origin xyz=0 0 -0.400 rpy=0 0 0 -> xyz=0 0 0 rpy=0 0 0; parent right_shank -> right_shank_ext
- joint right_knee_joint: origin xyz=0.400 0 0 rpy=0 0 0 -> xyz=0 0 0 rpy=0 0 0; parent right_thigh -> right_thigh_ext
