Commit message: fix(rehab): oscilatia gleznei -- castig 1.0, si de ce nu era amortizarea
Oscilatia din ziua 2 e reparata. Niciuna din cele doua cauze banuite nu era cea
reala; ambele au fost eliminate prin masurare, nu prin rationament.

IPOTEZA 1, INFIRMATA: 'comanda de viteza loveste clema'. Reconstruita viteza
COMANDATA la 93 Hz din datele reale (v = k * eroare, cu k si eroarea masurate):
maxim 0.42 rad/s dintr-o limita de 3.0369. Nu se apropie de clema. Ce se vedea fixat
pe limita era viteza ATINSA, retezata de Gazebo -- alt lucru.

IPOTEZA 2, INFIRMATA: 'amortizare insuficienta'. amort_glezna de la 2.0 la 20.0,
singura variabila schimbata: nicio diferenta masurabila.

CAUZA REALA: castigul. 15.0 -> 1.0 si oscilatia dispare complet.
  la 15.0 : schimbare de semn la FIECARE esantion (557/558), viteza fixata pe limita
            in 553/558, interval de pozitie 0.053 rad
  la  1.0 : interval de pozitie 0.00000 rad, zero esantioane pe limita
Explicatia care leaga totul: articulatia e comandata CINEMATIC. gz_ros2_control
scrie JointVelocityCmd = k * eroare si Gazebo o aplica drept constrangere de viteza,
nu drept cuplu. Nu exista nimic de invins, deci amortizarea nu are ce musca si
castigul mare doar suprareactioneaza. De aceea castigul MAI MIC urmareste MAI BINE:
treapta de 0.30 rad se aseaza la eroare 0.000, iar articulatiile necomandate nu mai
deriva deloc (la 15.0 aveau eroare reziduala 0.023).

CASTIG PER ARTICULATIE: nu e posibil. gz_ros2_control 1.2.17 expune doar un
position_proportional_gain GLOBAL; verificat direct in simbolurile bibliotecii, nu
exista forma per-articulatie. Raportat ca atare in loc sa fie simulat.

AMORTIZAREA ramane parametrizata per articulatie, cu valorile dinainte si statut
NEVERIFICAT (ca masele). Am pastrat-o desi nu ea a fost fixul, fiindca parametrizarea
a reparat un bug separat: ca <xacro:property>, 'amort_glezna:=99' era acceptat fara
eroare si IGNORAT IN TACERE. Sunt acum <xacro:arg>, deci suprascrierea chiar se
aplica. E a treia oara in doua zile cand o valoare pusa in locul gresit tace in loc
sa cada -- primele doua au fost position_proportional_gain in URDF si pe
controller_manager.

Consecinta scrisa in config si in README: cu comanda cinematica NU exista rejectie
de perturbatie. Cand modelul de pacient va aplica forte reale e nevoie de comanda in
EFORT, si acordarea se reia.

DUPA, exercitiul ankle_pump, toate patru verdictele monitorului:
  URMARIRE OK (max 0.000)  COERENTA OK (0.001)  CANALE OK  VITEZA OK (fara saturatie)
Suita: 18 teste, 0 esecuri.

Co-Authored-By: Claude Opus 5 <noreply@anthropic.com>

File: rehab_exo_description/urdf/rehab_exo.urdf.xacro (robot description, xacro)
@@ -69,4 +69,36 @@
   <xacro:property name="vi_genunchi" value="1.9732"/>
   <xacro:property name="vi_glezna"   value="3.0369"/>
+  <!-- AMORTIZARE SI FRECARE PE ARTICULATIE. Statut: NEVERIFICAT, acelasi ca masele.
+       Sunt necesare STABILITATII SIMULARII si INTERZISE concluziilor dinamice.
+       Documentul-sursa nu da coeficienti de amortizare (GAP 1, ca si masele).
+       De ce valori diferite si de ce glezna primeste mult mai mult: masurat pe
+       21 aug 2026, glezna intra in oscilatie la frecventa buclei de control, cu
+       schimbare de semn la FIECARE esantion si viteza fixata pe limita in 547 din
+       557 de esantioane, in timp ce soldul si genunchiul merg lin cu aceeasi
+       amortizare de 2.0. Cauza nu e clema de comanda: viteza COMANDATA reconstruita
+       (k * eroare) atinge maxim 0.42 rad/s dintr-o limita de 3.0369, deci nu se
+       apropie de ea. Cauza e raportul autoritate/inertie: 52 Nm de efort pe o
+       inertie de talpa de 0.00585 kg m2 dau ~8900 rad/s2, adica limita de viteza se
+       depaseste intr-un singur pas de simulare de 1 ms. Amortizarea de 2.0 e
+       neglijabila fata de asta.
+       Valorile de mai jos sunt ALESE prin masurare, nu derivate; vezi tabelul
+       inainte/dupa din raportul zilei 3.
+       Sunt ARGUMENTE, nu proprietati simple, si asta e deliberat: o proprietate NU
+       se poate suprascrie din linia de comanda, iar 'xacro ... amort_glezna:=99'
+       ar fi acceptat fara eroare si ignorat in tacere; a treia oara in aceeasi zi
+       cand o valoare pusa in locul gresit tace in loc sa cada. Ca argumente, se pot
+       balea si din launch. -->
+  <xacro:arg name="amort_sold"     default="2.0"/>
+  <xacro:arg name="amort_genunchi" default="2.0"/>
+  <xacro:arg name="amort_glezna"   default="2.0"/>
+  <xacro:arg name="frec_sold"      default="1.0"/>
+  <xacro:arg name="frec_genunchi"  default="1.0"/>
+  <xacro:arg name="frec_glezna"    default="1.0"/>
+  <xacro:property name="amort_sold"     value="$(arg amort_sold)"/>
+  <xacro:property name="amort_genunchi" value="$(arg amort_genunchi)"/>
+  <xacro:property name="amort_glezna"   value="$(arg amort_glezna)"/>
+  <xacro:property name="frec_sold"      value="$(arg frec_sold)"/>
+  <xacro:property name="frec_genunchi"  value="$(arg frec_genunchi)"/>
+  <xacro:property name="frec_glezna"    value="$(arg frec_glezna)"/>
   <xacro:arg name="controllers"
              default="$(find rehab_exo_description)/config/controllers.yaml"/>
@@ -285,5 +317,5 @@
     <axis xyz="0 -1 0"/>
     <limit lower="${sold_lo}" upper="${sold_hi}" effort="${ef_sold}" velocity="${vi_sold}"/>
-    <dynamics damping="2.0" friction="1.0"/>
+    <dynamics damping="${amort_sold}" friction="${frec_sold}"/>
   </joint>
   <link name="${side}_thigh">
@@ -346,5 +378,5 @@
     <axis xyz="0 1 0"/>
     <limit lower="${gen_lo}" upper="${gen_hi}" effort="${ef_genunchi}" velocity="${vi_genunchi}"/>
-    <dynamics damping="2.0" friction="1.0"/>
+    <dynamics damping="${amort_genunchi}" friction="${frec_genunchi}"/>
   </joint>
   <link name="${side}_shank">
@@ -397,5 +429,5 @@
     <axis xyz="0 -1 0"/>
     <limit lower="${gle_lo}" upper="${gle_hi}" effort="${ef_glezna}" velocity="${vi_glezna}"/>
-    <dynamics damping="2.0" friction="1.0"/>
+    <dynamics damping="${amort_glezna}" friction="${frec_glezna}"/>
   </joint>
   <link name="${side}_foot">

Commit message: fix(rehab): alinierea pacient-masina, gasita in capturile RViz
CE SE VEDEA in inspectia vizuala: picioarele pacientului (cilindrii portocaliu si
albastru) porneau vizibil din alt loc decat trunchiul lui. Masurat: bazinul
pacientului era cu 0.270 m in spate si 0.060 m sub axa soldului masinii.

DE CE CONTEAZA MAI MULT DECAT PARE. Ca axa articulatiei masinii sa treaca prin
articulatia omului nu e o chestiune de aspect: e cerinta de baza a oricarui
exoschelet. Daca nu coincid, orice unghi comandat produce alt unghi la pacient, plus
o forta de forfecare pe segment. Un model care le lasa decalate ar da cifre de
"unghi de sold" care nu sunt unghiul de sold al nimanui.

Niciun test nu o prindea, si merita spus de ce: nu incalca topologia, nu incalca
limitele, nu atinge podeaua. Era invizibila pentru tot ce construisem, si vizibila
imediat pentru un om care se uita la ecran. E argumentul pentru care poarta vizuala
exista.

CAUZA nu era omul, ci ADANCIMEA SCAUNULUI. La 0.460 m axa soldului cadea la marginea
din fata a pernei, adica la 0.27 m in fata bazinului. Perna insa sustine DOAR bazinul:
coapsa e purtata de modulul mecanic [Fig 2.4, reper 2], nu de scaun. Adancimea trece
la 0.300 m, spatarul se aseaza derivat la marginea din spate, si bazinul pacientului
primeste exact offsetul articulatiei de sold.
Rezultat: decalaj 0.0000 / 0.0000 m. Spatele pacientului la 0.045 m de spatar.

Perna, spatarul si pozitia pacientului nu mai au cote literale: ies din cote_derivate,
ca restul.

ASERTAT in test_podea, ca sa nu se mai poata strica in tacere: pe ambele picioare, axa
soldului masinii trebuie sa treaca prin bazinul pacientului, la 1e-9.

Suita: 28 de teste, 0 esecuri, 1 skip enumerat.

Co-Authored-By: Claude Opus 5 <noreply@anthropic.com>

File: rehab_exo_description/urdf/rehab_exo.urdf.xacro (robot description, xacro)
@@ -235,5 +235,5 @@
     <visual>
       <origin xyz="0.0000 0.0000 0.0000" rpy="0 0 0"/>
-      <geometry><box size="0.4600 0.4600 0.0700"/></geometry>
+      <geometry><box size="${g_scaun_lungime} 0.4600 ${g_scaun_grosime}"/></geometry>
       <material name="cushion"/>
     </visual>
@@ -270,10 +270,10 @@
     <collision>
       <origin xyz="0.0000 0.0000 0.0000" rpy="0 0 0"/>
-      <geometry><box size="0.4600 0.4600 0.0700"/></geometry>
+      <geometry><box size="${g_scaun_lungime} 0.4600 ${g_scaun_grosime}"/></geometry>
     </collision>
   </link>
   <joint name="seat_to_back" type="fixed">
     <parent link="seat_link"/><child link="backrest_link"/>
-    <origin xyz="-0.235 0 0.02" rpy="0 -0.21 0"/>
+    <origin xyz="${-g_scaun_lungime/2} 0 0.02" rpy="0 -0.21 0"/>
   </joint>
   <link name="backrest_link">
@@ -305,34 +305,39 @@
   <joint name="seat_to_human" type="fixed">
     <parent link="seat_link"/><child link="human_torso"/>
-    <origin xyz="-0.04 0 0.035" rpy="0 0 0"/>
+    <!-- ALINIEREA PACIENT-MASINA. Bazinul pacientului se pune EXACT pe axa soldului
+         masinii, cu acelasi offset ca articulatia de sold. E cerinta de baza a
+         oricarui exoschelet, si pana pe 22 aug era incalcata cu 0.27 m pe x si
+         0.06 m pe z: in RViz se vedea ca picioarele pacientului porneau din alt loc
+         decat trunchiul lui. -->
+    <origin xyz="${g_sold_x - g_scaun_centru_x} 0 ${g_sold_inaltime - g_scaun_centru_z}" rpy="0 0 0"/>
   </joint>
   <link name="human_torso">
     <inertial>
-      <origin xyz="0.0000 0.0000 0.2800" rpy="0 0 0"/>
+      <origin xyz="-0.1000 0.0000 0.2800" rpy="0 0 0"/>
       <mass value="32.000"/>
       <inertia ixx="1.029333" ixy="0" ixz="0" iyy="0.874667" iyz="0" izz="0.461867"/>
     </inertial>
     <visual>
-      <origin xyz="0.0000 0.0000 0.2800" rpy="0 0 0"/>
+      <origin xyz="-0.1000 0.0000 0.2800" rpy="0 0 0"/>
       <geometry><box size="0.2400 0.3400 0.5200"/></geometry>
       <material name="cloth"/>
     </visual>
     <visual>
-      <origin xyz="0.0100 0.0000 0.6650" rpy="0 0 0"/>
+      <origin xyz="-0.0900 0.0000 0.6650" rpy="0 0 0"/>
       <geometry><sphere radius="0.1050"/></geometry>
       <material name="skin"/>
     </visual>
     <visual>
-      <origin xyz="0.0100 0.0000 0.5550" rpy="0 0 0"/>
+      <origin xyz="-0.0900 0.0000 0.5550" rpy="0 0 0"/>
       <geometry><cylinder radius="0.0450" length="0.0700"/></geometry>
       <material name="skin"/>
     </visual>
     <visual>
-      <origin xyz="0.0000 0.2050 0.4000" rpy="0.15 0 0"/>
+      <origin xyz="-0.1000 0.2050 0.4000" rpy="0.15 0 0"/>
       <geometry><cylinder radius="0.0450" length="0.2600"/></geometry>
       <material name="cloth"/>
     </visual>
     <visual>
-      <origin xyz="0.0000 -0.2050 0.4000" rpy="-0.15 0 0"/>
+      <origin xyz="-0.1000 -0.2050 0.4000" rpy="-0.15 0 0"/>
       <geometry><cylinder radius="0.0450" length="0.2600"/></geometry>
       <material name="cloth"/>
@@ -359,5 +364,5 @@
     </visual>
     <collision>
-      <origin xyz="0.0000 0.0000 0.2800" rpy="0 0 0"/>
+      <origin xyz="-0.1000 0.0000 0.2800" rpy="0 0 0"/>
       <geometry><box size="0.2400 0.3400 0.5200"/></geometry>
     </collision>

Commit message: feat(rehab): seat band re-justified in B-prim + supervisor update
Banda transportata mecanic (minus 65 pana la 0) e MOARTA oficial. Continutul nou e
construit de la zero in termeni B-prim, cu derivarea aratata in IPOTEZE_LIMITE.md.

SURSA 1, FORMA. Citatul verbatim din [PDF p.7]: blocul 204 se misca INTRE inelele 201
si 208, iar extinderea lui 208 REDUCE cursa. Fapt: banda de sezut e o SUBMULTIME care
pastreaza un capat. Presupunere NUMITA ca atare: textul nu spune CARE capat, iar noi
presupunem ca repausul (B-prim zero) apartine benzii de antrenament in sezut, fiindca
altfel dispozitivul n-ar putea antrena chiar in postura in care sta. De aici 0..X.
Proximity-urile rastoarna sau confirma presupunerea la prima vizita.

SURSA 2, CAPATUL DE SUS. Argumentul pernei, pe care il banuisem, e INFIRMAT prin
masurare si consemnat ca respins ca sa nu fie reinventat: perna se termina exact la
axa soldului, coapsa pleaca inainte pe langa ea, si nici la minus 30 de grade nu
exista contact. Ce margineste efectiv: in jos invariantul podelei (argumentul D1), in
sus interferenta coapsa-trunchi. X = 25 grade mecanic, adica circa 115 grade de flexie
anatomica -- marginea conservatoare pentru populatia de reabilitare. Clasa
IPOTEZA-ANTROPO.

SURSA 3, banda 65-80 LLR-Ro: NEUTILIZABILA, citata ca sa nu fie recuperata din
greseala. 65 e o LATIME, nu o pozitie; 65-80 dintr-un total de 90 nu e o reducere,
deci contrazice "the motion space is small"; iar sursa nu are referinta verificabila.

IPOTEZA CONCURENTA, scrisa si nefolosita: valorile URDF-ului livrat (-25.78..+40.11
fata de un zero declarat SEZUT) nu au sursa, dar daca autorul lor cunostea
dispozitivul, banda reala ar cobori usor sub orizontala si ar urca spre 40, nu spre
25. Proximity-urile transeaza intre cele doua.

DEFECT GASIT DE PROBA NUMERICA, si reparat: verdict_comutare verifica acum limitele
MECANICE ale posturii-tinta, nu pragurile electrice. Cu praguri, comutarea era
refuzata chiar din POSTURA_INITIALA (sold 0 e sub pragul electric de 5 grade), adica
serviciul era inutilizabil taman din pozitia in care dispozitivul sta. Intrebarea
"pot trece la postura asta" e despre legalitatea pozitiei in noul set, nu despre marja
de declansare; dupa comutare, o articulatie intre limita mecanica si prag ramane pur
si simplu NEARMATA, comportamentul deja proiectat pentru pornire. Selftestul are acum
si controlul care arata ca pe praguri aceeasi pozitie ar fi fost refuzata.

DOVEZI NUMERICE (praguri electrice: culcat sold 5..85, sezut 5..20):
  POSTURA_INITIALA, sold 0   NEARMAT, 0 declansari
  dupa intrare la 12 grade   ARMAT
  la 22 grade                2 declansari, "0.3840 rad a depasit pragul max 0.3491"
  comutare din 0 / 12 / 25   PERMISA
  comutare din 60            refuzata, cu articulatia si valoarea in mesaj

ASERTIA DIN test_podea A FOST INVERSATA DELIBERAT, exact cum prevedea comentariul ei:
cat timp banda era transportata, testul cerea sa PICE; re-justificata, ea descrie
configuratii reale si trebuie sa TREACA. Inversarea e vizibila in fisier, nu tacuta.
Baleiere: 200 de configuratii legale si in sezut, cel mai jos punct +0.0307 m.
Adaugat si ca sezutul trebuie sa fie SUBMULTIME care pastreaza capatul de jos.

Invariantele permanente re-rulate dupa atingerea limitelor: FK 74 verificari verzi,
podea 411 verificari verzi. Suita: 28 de teste, 0 esecuri.

Co-Authored-By: Claude Opus 5 <noreply@anthropic.com>

File: rehab_exo_description/urdf/rehab_exo.urdf.xacro (robot description, xacro)
@@ -60,15 +60,21 @@
   <xacro:property name="sold_min_deg"      value="0"/>
   <xacro:property name="sold_max_deg"      value="90"/>
-  <!-- BANDA DE SEZUT: TRANSPORTATA mecanic din conventia veche prin aceeasi mapare
-       ca restul (se scad 90 de grade din 25..90), NU validata. Rezultatul cade
-       integral SUB orizontala, deci e geometric imposibil, si tocmai asta e dovada
-       ca plasarea veche era gresita. Se pastreaza in forma transportata ca sa nu
-       ramana nimic in doua conventii, si se REJUDECA separat (punctul 5), impreuna
-       cu fraza din document: "in sitting position, the motion space of the hip joint
-       is small". Pana atunci: postura sezut produce deliberat un model care PICA
-       invariantul podelei, iar test/test_podea.py aserteaza exact acest lucru.
-       Implicitul ramane culcat. -->
-  <xacro:property name="sold_sezut_min_deg" value="-65"/>
-  <xacro:property name="sold_sezut_max_deg" value="0"/>
+  <!-- BANDA DE POSTURA SEZUT, RE-JUSTIFICATA (nu convertita) pe 22 aug 2026.
+       Banda transportata mecanic (minus 65 pana la 0) a MURIT: cadea integral sub
+       orizontala, deci era imposibila geometric. Continutul de aici e construit de la
+       zero, in termeni B-prim. Derivarea completa, cu ce a fost respins si de ce, sta
+       in urdf/IPOTEZE_LIMITE.md; pe scurt:
+         FORMA, din [PDF p.7]: blocul 204 se misca INTRE inelele 201 si 208, iar
+         extinderea lui 208 reduce cursa. Deci banda de sezut e o submultime care
+         PASTREAZA UN CAPAT din cursa completa. Textul nu spune CARE capat; se
+         presupune, explicit, ca repausul (B-prim zero) apartine benzii de
+         antrenament in sezut. De aici forma 0..X.
+         CAPATUL DE SUS, ANTROPO: la spatar vertical, coapsa ridicata intra in
+         trunchi. X = 25 grade mecanic inseamna circa 115 grade de flexie anatomica,
+         marginea conservatoare pentru populatia de reabilitare.
+       Clasa: IPOTEZA-ANTROPO. Pozitiile proximity-urilor o inchid definitiv; item pe
+       agenda vizitei. -->
+  <xacro:property name="sold_sezut_min_deg" value="0"/>
+  <xacro:property name="sold_sezut_max_deg" value="25"/>
   <xacro:property name="genunchi_min_deg"  value="0"/>
   <xacro:property name="genunchi_max_deg"  value="140"/>

Commit message: docs(rehab): exercise inventory + full smoke table
INVENTARUL celor 12 exercitii: articulatiile care se misca EFECTIV (derivate din
esantionarea traiectoriei, nu din nume), numarul de puncte, durata, repetarile si
comenzile de rulare.

SMOKE PE TOATE 12, cu supervizor activ, intr-o singura sesiune Gazebo: trimise pe
rand pe /exercise_cmd, cu verdictele calculate de ACELEASI functii pure ca monitorul.
Trei exercitii pica pe URMARIRE (hip_alternating 1.1145 rad, hip_hold 1.1935,
leg_wave 0.2335) si toate trei din aceeasi cauza.

DEFECT DESCHIS, raportat cu cifre si NU reparat tacit, fiindca e o decizie despre
stratul de siguranta:

Pragul electric sta la 5 grade inauntru fata de limita mecanica la AMBELE capete, dar
exercitiile folosesc legitim capatul de jos al ferestrei documentate: soldul coboara
la 0.00 grade (repausul insusi), genunchiul la 4.06. Deci orice exercitiu care revine
la repaus trece sub prag, declanseaza, iar supervizorul FACE LATCH si tine
articulatia pana la finalul sesiunii. De aici cele trei esecuri de urmarire: nu e
geometrie, nu e acordare, e un joint tinut de propriul supervizor.
Masurat: 4 declansari, toate pe capatul min, intre 0.0664 si 0.0781 rad.
Cauza de fond e ordonarea straturilor: corect ar fi mecanic > electric > software,
adica traiectoriile INAUNTRUL ferestrei electrice; la noi ele ating capatul mecanic.
Doua rezolvari aparabile sunt scrise in README; alegerea e a omului.

BUG REPARAT PE DRUM, gasit in timp ce cautam cauza: coloana verticala a soldului,
adaugata de mine la P1, avea si COLIZIUNE. Ea urca exact pana la axa soldului, iar
coapsa are grosime, deci aveau volum comun permanent langa pivot (x in [0, 0.07],
z in [0.689, 0.729]); cum base_link si coapsa nu sunt parinte-copil, Gazebo le
ciocnea. Coloana devine element VIZUAL: bracketul real are un decupaj de gabarit in
jurul pivotului, dar geometria lui nu e in document, iar o coliziune inventata e mai
rea decat absenta ei.
Nu era insa cauza blocajului observat: dupa fix soldul urmarea perfect comenzi
directe (0.2 pana la 1.3 rad, eroare 0.0000), ceea ce a si aratat ca vinovatul e
latch-ul supervizorului.

O NOTA DE ONESTITATE despre propria mea proba: coloana de declansari din tabelul de
smoke subnumara, fiindca probeul se abona DUPA ce latch-ul pornise. Cifra corecta,
luata din log, e 4. Tabelul o spune explicit in loc s-o corectez in tacere.

Suita: 30 de teste, 0 esecuri.

Co-Authored-By: Claude Opus 5 <noreply@anthropic.com>

File: rehab_exo_description/urdf/rehab_exo.urdf.xacro (robot description, xacro)
@@ -213,9 +213,14 @@
         <material name="frame_gri"/>
       </visual>
-      <collision>
-        <origin xyz="${g_sold_x} ${sy * g_sold_y} ${(g_placa_grosime + g_sold_inaltime)/2}"
-                rpy="0 0 0"/>
-        <geometry><box size="0.1400 0.1000 ${g_sold_inaltime - g_placa_grosime}"/></geometry>
-      </collision>
+      <!-- FARA COLIZIUNE, si asta nu e o scurtatura. Coloana urca EXACT pana la axa
+           soldului, iar coapsa are grosime, deci cele doua au un volum comun
+           permanent langa pivot: x in [0, 0.07] si z in [0.689, 0.729]. Cum
+           base_link si coapsa nu sunt parinte-copil, Gazebo le ciocneste si
+           BLOCHEAZA soldul complet; masurat pe 22 aug, referinta urca la 1.3464 rad
+           si masuratul ramane la 0.0000 pe toata durata exercitiului.
+           Bracketul real are un decupaj de gabarit in jurul pivotului, dar geometria
+           lui nu e in document (acelasi GAP ca restul cotelor). Pana cand exista,
+           coloana ramane element VIZUAL: prezenta ei in coliziuni ar fi o
+           constrangere INVENTATA, mai rea decat absenta ei. -->
     </xacro:macro>
     <xacro:coloana_sold sy="1"/>
