Commit message: fix(rehab): D3 opritorul sub repaus -- soldul se misca, 12/12
DECIZIA A. Fereastra soldului devine -2..88: latimea documentata de 90 se pastreaza,
se muta PLASAREA, care a fost mereu IPOTEZA. POSTURA_INITIALA ramane la 0, deci ancora
lui D1 e intacta: repausul e tinut de CONTROL, iar opritorul de la -2 il prinde pasiv,
ca pe masina reala. Banda de sezut isi urmeaza capatul de jos la -2 si isi pastreaza
capatul ANTROPO la 25. Inaltimea talpii se re-alege prin propriul ei criteriu, de la
0.230 la 0.250, ca invariantul podelei sa redevina verde: masurat, la 0.230 cu sold_min
-2 cel mai jos punct cadea la +0.0127, sub marja de 0.030.

REZULTAT, re-smoke pe toate 12 cu eroarea MAXIMA continua si supervizor activ:
12 din 12, 0 declansari, cea mai mare eroare din tot tabelul 0.0152 rad (0.87 grade).
Inainte, cele patru exercitii de sold lasau articulatia complet nemiscata, cu eroarea
egala cu amplitudinea comandata (1.3464, 1.2342, 1.1220, 0.7853).

TREI TESTE MI-AU SPUS CA PREMISELE LOR S-AU SCHIMBAT, si fiecare exact cum fusese
scris sa faca. test_descriere si test_supervizor codificau fereastra 0..90.
Iar asertia "premisa testului: minimul soldului e 0.0 (daca se schimba, revizuieste)"
si-a facut treaba literal: testul de pornire-pe-margine se rescrie acum pe GENUNCHI,
care isi pastreaza minimul la 0 si ramane deci cazul real de armare.

CONSECINTA BUNA A LUI D3: soldul nu mai sta pe capat, deci se poate arma chiar de la
pornire -- e supravegheat imediat, nu dupa prima intrare in zona.
CONSECINTA DE SEPARAT, scrisa in D3: rezerva de repaus (2 grade) e EXACT cat banda de
armare (2 grade), deci starea de armare la repaus sta la granita si poate bascula cu
zgomotul solverului. Se aserteaza proprietatea ROBUSTA (nu declanseaza), nu eticheta
de stare, care aici nu e determinista. Cele doua cifre nu ar trebui sa fie egale.

ANEXA (i), articulatiile prismatice: verificate empiric, NU presupuse -- si
rationamentul meu gravitational a fost CONTRAZIS. Comandate sa se mute de la repaus,
seat_lift a coborat pana pe celalalt capat in loc sa se opreasca unde i s-a cerut, iar
cele patru reglaje nu s-au miscat deloc. Nu sunt deci exemptii dovedite, ci items
DESCHISE cu statut scris; cauza nu e stabilita si poate fi alta decat mecanismul
soldului. Exercitiile nu le folosesc, deci nu ating cele 12.

D3 in DECIZII.md, cu cele trei linii de convergenta: principiul opritorului (acelasi
ca D2), prima confirmare partiala a ipotezei concurente din registru (URDF-ul livrat
avea semiplanul negativ, iar fizica il cere), si diferenta de modelare acum inteleasa
(real: coapsa se odihneste pe perna, care preia sarcina; model: perna se termina la
axa, deci coapsa atarna in articulatie si incarca limita cum masina reala n-o incarca).

NOTA TEHNICA in material_teza, cu versiunile exacte (Gazebo Sim 8.11.0,
gz_ros2_control 1.2.17): comanda de viteza vs constrangerea de limita, cu
discriminatorul care conteaza pentru altii -- nu tipul articulatiei sau controllerul,
ci DIRECTIA in care gravitatia impinge fiecare articulatie fata de limita pe care se
odihneste.

AGENDA VIZITEI, pe primul loc acum: INALTIMEA SCAUNULUI. Prin alegeri INVARIANT
succesive axa soldului a urcat de la 0.60 la 0.749 m si scaunul la 0.689 -- inaltime
de taburet, nu de scaun de reabilitare. De ea atarna tot lantul vertical.

Suita: 36 de teste, 0 esecuri. Invariantele permanente verzi: FK 74, podea 411.

Co-Authored-By: Claude Opus 5 <noreply@anthropic.com>

File: rehab_exo_description/urdf/rehab_exo.urdf.xacro (robot description, xacro)
@@ -58,6 +58,13 @@
        IPOTEZA (GAP 4) si a fost RE-DERIVATA la D1: repausul e coapsa orizontala si
        cursa merge in sus, fiindca in jos piciorul ar trece prin podea. -->
-  <xacro:property name="sold_min_deg"      value="0"/>
-  <xacro:property name="sold_max_deg"      value="90"/>
+  <!-- MINUS 2 GRADE, nu zero (decizia A, 22 aug). Repausul soldului e coapsa
+       orizontala, adica 0; daca limita mecanica ar fi tot acolo, articulatia s-ar
+       odihni PE opritor. Masurat: in acea configuratie constrangerea de limita din
+       solver tine articulatia si comanda de viteza a lui gz_ros2_control nu o mai
+       poate elibera. Pe masina reala opritorul sta SUB pozitia de repaus: motorul
+       tine pozitia, stopul o prinde pasiv. Latimea documentata de 90 de grade se
+       pastreaza; fereastra devine -2..88. Vezi DECIZII.md, D3. -->
+  <xacro:property name="sold_min_deg"      value="-2"/>
+  <xacro:property name="sold_max_deg"      value="88"/>
   <!-- BANDA DE POSTURA SEZUT, RE-JUSTIFICATA (nu convertita) pe 22 aug 2026.
        Banda transportata mecanic (minus 65 pana la 0) a MURIT: cadea integral sub
@@ -75,5 +82,9 @@
        Clasa: IPOTEZA-ANTROPO. Pozitiile proximity-urilor o inchid definitiv; item pe
        agenda vizitei. -->
-  <xacro:property name="sold_sezut_min_deg" value="0"/>
+  <!-- Capatul de JOS se imparte cu fereastra completa, deci urmeaza si el la -2
+       (D3): structura din P2.1 spune ca banda de sezut e o SUBMULTIME care pastreaza
+       un capat, iar acela e cel de jos. Capatul de SUS ramane cel ANTROPO, 25 grade,
+       neatins de aceasta decizie. -->
+  <xacro:property name="sold_sezut_min_deg" value="-2"/>
   <xacro:property name="sold_sezut_max_deg" value="25"/>
   <xacro:property name="genunchi_min_deg"  value="0"/>
