Commit message: feat(rehab): anatomic zero B + documented ROM + dual posture (F1b)
M1 din ziua task-force. Conventia articulara trece de la zeroul mostenit
(zero = SEZUT, declarat in antetul URDF-ului livrat) la ZEROUL ANATOMIC, decizia B
din registrul de pe 18 aug. Cursele totale devin cele documentate.

CONVENTIA NOUA, plan sagital:
  sold     0 = coapsa colineara cu trunchiul, POZITIV = FLEXIE
  genunchi 0 = gamba colineara cu coapsa,     POZITIV = FLEXIE
  glezna   0 = talpa perpendiculara pe gamba, POZITIV = DORSIFLEXIE
Maparea NU a fost presupusa, ci derivata prin cinematica directa pe URDF-ul livrat:
la q=0 vechi coapsa arata spre +X (orizontal) si gamba spre -Z (vertical), iar
trunchiul (human_torso, rpy 0 0 0) e pe +Z. Rezulta hip_nou = hip_vechi + 90 grade.
La genunchi, FK arata ca unghiul vechi crestea spre EXTENSIE (gamba se rotea de la -Z
spre +X), deci in conventia anatomica semnul SE INVERSEAZA: knee_nou = 90 - knee_vechi,
materializat prin axa (0 1 0) in loc de (0 -1 0) plus rotatia originii.

CURSELE [PDF Tabel 3.1, p.10-11]: sold 90, genunchi 140, glezna 70 grade.
IMPARTIREA min/max ramane GAP 4: parametri xacro in grade, cu suma asertata egala cu
cursa documentata, si urdf/IPOTEZE_LIMITE.md care da ipoteza si rationamentul per
articulatie. Nicio ipoteza nu e prezentata ca fapt.

POSTURA: postura:=culcat|sezut. In sezut, inelul de oprire (reper 208, PDF p.7) reduce
mecanic cursa soldului la 25..90 grade. Testul verifica explicit ca postura atinge
NUMAI soldul.

ECHIVALENTA, dovedita programatic (test/test_conventie.py, 255 verificari): pozitia si
orientarea talpii, calculate din descrierea veche la unghiul vechi si din cea noua la
unghiul convertit, pe 62 de configuratii x 2 picioare. Abatere maxima 2.5e-16 m si
4.4e-16 pe rotatie -- epsilon de masina. Control negativ: o mapare fara inversarea
semnului la genunchi da 0.599 m abatere, deci testul chiar poate pica.

TRAIECTORIILE: conversie programatica, NU manuala, si NU uniforma -- iar asta e
descoperirea zilei. Genunchi si glezna: offset (cu inversare la genunchi), unghi FIZIC
identic. Soldul: RE-DERIVAT. Motivul, masurat: cursa veche a soldului, exprimata
anatomic, e 64.22..130.11 grade -- sold permanent flectat, peste flexia umana normala
(~120-125) -- si NU incape in cei 90 documentati; 132 de puncte ieseau, cu depasire
maxima de 34.4 grade. Nicio fereastra de 90 de grade nu ar fi salvat-o, deci nicio
alegere de split. Limitele vechi erau placeholdere fara sursa; documentul are
prioritate. Punctele pastreaza FRACTIA din cursa disponibila, adica forma
exercitiului, nu unghiul absolut. test/test_traiectorii.py verifica cele DOUA
invariante separat: 1908 valori, 2404 verificari.

A doua descoperire, tot prin test: starea initiala a programului era implicit
{toate 0.0}, ceea ce in conventia veche insemna FIZIC sezut. Lasata asa, ar fi devenit
culcat drept -- alta miscare, fara ca nimic sa semnaleze. E acum POSTURA_INITIALA,
declarata explicit si convertita.

Selftestul descrierii cere acum si ca CURSA TOTALA sa fie cea documentata, oricare ar
fi impartirea. README rescris; conventia veche trimite la attic/.

colcon build curat de la zero: OK. colcon test: 6 teste, 0 erori, 0 esecuri.

File: rehab_exo_description/urdf/rehab_exo.urdf.xacro (robot description, xacro)
@@ -9,4 +9,51 @@
        ou si gaina. CMake paseaza calea de instalare; generarea manuala foloseste
        implicitul, care merge dupa ce pachetul a fost instalat macar o data. -->
+  <xacro:arg name="postura" default="culcat"/>
+  <xacro:property name="postura" value="$(arg postura)"/>
+  <!-- ============ CONVENTIA ARTICULARA: ZERO ANATOMIC ============
+       Decizia din registru, 18 aug, varianta B. Conventia veche (zero = SEZUT)
+       s-a pensionat; e in attic/rehab_exo.urdf.livrat.
+       Zero pentru fiecare articulatie, in plan sagital:
+         sold     0 = coapsa colineara cu trunchiul (culcat drept). POZITIV = FLEXIE
+                  (coapsa se ridica spre piept).
+         genunchi 0 = gamba colineara cu coapsa (extensie completa). POZITIV = FLEXIE
+                  (calcaiul se apropie de sezut).
+         glezna   0 = talpa perpendiculara pe gamba (neutru). POZITIV = DORSIFLEXIE
+                  (varful piciorului urca).
+       Trunchiul e pe +Z (verificat pe geometria human_torso, cutie 0.24x0.34x0.52
+       cu rpy 0 0 0), deci coapsa la zero anatomic arata spre -Z.
+       ATENTIE la genunchi: in conventia veche unghiul CRESTEA spre extensie
+       (verificat prin cinematica directa: gamba se rotea de la -Z spre +X). In
+       conventia noua creste spre FLEXIE. Inversarea de semn e materializata prin
+       axa (0 1 0) in loc de (0 -1 0), plus rotatia de origine. Echivalenta fizica
+       e dovedita programatic in test/test_conventie.py, nu prin citire.
+       CURSELE TOTALE sunt cele documentate [PDF Tabel 3.1, p.10-11]:
+         sold 90 grade, genunchi 140 grade, glezna 70 grade.
+       IMPARTIREA min/max NU e in document (GAP 4): valorile de mai jos sunt
+       IPOTEZE LOCALE, motivate in urdf/IPOTEZE_LIMITE.md. Suma lor e asertata
+       egala cu cursa documentata, deci ipoteza poate fi schimbata fara sa se
+       piarda fidelitatea fata de document.
+       ============================================================ -->
+  <xacro:property name="rom_sold_deg"      value="90"/>
+  <xacro:property name="rom_genunchi_deg"  value="140"/>
+  <xacro:property name="rom_glezna_deg"    value="70"/>
+  <xacro:property name="sold_min_deg"      value="0"/>
+  <xacro:property name="sold_max_deg"      value="90"/>
+  <xacro:property name="sold_sezut_min_deg" value="25"/>
+  <xacro:property name="genunchi_min_deg"  value="0"/>
+  <xacro:property name="genunchi_max_deg"  value="140"/>
+  <xacro:property name="glezna_min_deg"    value="-35"/>
+  <xacro:property name="glezna_max_deg"    value="35"/>
+  <!-- Postura schimba DOAR limita inferioara a soldului: in sezut, inelul de
+       oprire (reper 208, PDF p.7) reduce mecanic cursa. IPOTEZA LOCALA. -->
+  <xacro:property name="sold_lo_deg"
+                  value="${sold_sezut_min_deg if postura == 'sezut' else sold_min_deg}"/>
+  <xacro:property name="d2r" value="${pi / 180.0}"/>
+  <xacro:property name="sold_lo" value="${sold_lo_deg * d2r}"/>
+  <xacro:property name="sold_hi" value="${sold_max_deg * d2r}"/>
+  <xacro:property name="gen_lo"  value="${genunchi_min_deg * d2r}"/>
+  <xacro:property name="gen_hi"  value="${genunchi_max_deg * d2r}"/>
+  <xacro:property name="gle_lo"  value="${glezna_min_deg * d2r}"/>
+  <xacro:property name="gle_hi"  value="${glezna_max_deg * d2r}"/>
   <xacro:arg name="controllers"
              default="$(find rehab_exo_description)/config/controllers.yaml"/>
@@ -210,7 +257,7 @@
   <joint name="${side}_hip_joint" type="revolute">
     <parent link="seat_link"/><child link="${side}_thigh"/>
-    <origin xyz="0.160 ${sy * 0.260} 0.035" rpy="0 0 0"/>
+    <origin xyz="0.160 ${sy * 0.260} 0.035" rpy="0 ${pi/2} 0"/>
     <axis xyz="0 -1 0"/>
-    <limit lower="-0.45" upper="0.7" effort="120.0" velocity="2.0"/>
+    <limit lower="${sold_lo}" upper="${sold_hi}" effort="120.0" velocity="2.0"/>
     <dynamics damping="2.0" friction="1.0"/>
   </joint>
@@ -271,7 +318,7 @@
   <joint name="${side}_knee_joint" type="revolute">
     <parent link="${side}_thigh_ext"/><child link="${side}_shank"/>
-    <origin xyz="0 0 0" rpy="0 0 0"/>
-    <axis xyz="0 -1 0"/>
-    <limit lower="0.0" upper="1.75" effort="120.0" velocity="2.0"/>
+    <origin xyz="0 0 0" rpy="0 ${-pi/2} 0"/>
+    <axis xyz="0 1 0"/>
+    <limit lower="${gen_lo}" upper="${gen_hi}" effort="120.0" velocity="2.0"/>
     <dynamics damping="2.0" friction="1.0"/>
   </joint>
@@ -324,5 +371,5 @@
     <origin xyz="0 0 0" rpy="0 0 0"/>
     <axis xyz="0 -1 0"/>
-    <limit lower="-0.6" upper="0.6" effort="120.0" velocity="2.0"/>
+    <limit lower="${gle_lo}" upper="${gle_hi}" effort="120.0" velocity="2.0"/>
     <dynamics damping="2.0" friction="1.0"/>
   </joint>

Commit message: feat(rehab): documented effort/velocity limits with provenance
M2. Cifrele vechi de efort si viteza (120 Nm pe toate revolute, 2.0 rad/s pe toate,
300/500 Nm si 0.03/0.05 pe prismatice) nu aveau nicio sursa. Acum fiecare limita de pe
articulatiile revolute e DERIVATA din documentatie, cu formula si proveniente.

NUCLEU PUR: scripts/spec_derivate.py, 27 de verificari in selftest, fara ROS si fara
fisiere. urdf/SPEC_DERIVATE.md se GENEREAZA din el, deci documentul nu poate devia de
cod.

FORMULE
  viteza [rad/s] = (rpm_motor / 60) * 2*pi / raport_total
  efort  [Nm]    = min(cuplu_motor * raport_total * eta, cuplu_nominal_reductor)

REZULTAT
  articulatie  raport   rpm   viteza[rad/s]  efort[Nm]  limitat de
  sold         245.45   3700  1.5786         176.7      motorul
  genunchi     196.36   3700  1.9732         141.4      motorul
  glezna       100.00   1500  1.5708          52.0      reductorul
Observatie de proiectare: la sold si genunchi motorul limiteaza (176.7 din 345
disponibili la SHG-40, 141.4 din 178 la SHG-32); la glezna limiteaza reductorul.

IPOTEZE, toate declarate si parametrizate
 - eta = 0.80 (randamentul lantului curea + armonic). La glezna exista un PRAG calculat:
   eta = 52/(0.706*100) = 0.7365. Peste el limiteaza reductorul, sub el motorul. Ipoteza
   de 0.80 e PESTE prag, deci daca randamentul real e mai mic, efortul gleznei scade sub
   52 Nm. Pragul si ambele ramuri sunt asertate in selftest.
 - turatia TBM(S)-6025 = 1500 rpm: nu apare in partea citita a foii. Afecteaza DOAR
   viteza gleznei, nu efortul.
 - motor sold/genunchi: lista de componente numeste SMP8024B, foaia anexata e pentru
   SMP8048. Se folosesc cifrele foii; discrepanta ramane VIZIBILA in date (campurile
   'nume' si 'foaie' difera, si un selftest cere sa difere). DE CONFIRMAT FIZIC.

DOUA ASERTTII CORECTATE PE DRUM, ambele scriau o asteptare in loc de un fapt:
 - 'la glezna eta nu are efect' era falsa la eta=0.5, unde motorul chiar preia
   limitarea. Inlocuita cu pragul de basculare si ambele ramuri.
 - 'glezna e mai rapida decat soldul' era o ASTEPTARE: viteza ei depinde de rpm-ul
   presupus, si cu 1500 rpm iese aproape egala cu soldul. Inlocuita cu relatia care
   chiar decurge din rapoarte: la acelasi rpm, viteza scaleaza invers cu raportul
   (2.4545 ori).

LEGATURA URDF <-> SURSA: selftestul descrierii recalculeaza acum efortul si viteza din
nucleul pur si le confrunta cu URDF-ul GENERAT; plus o asertie ca cifrele vechi fara
sursa (120.0 / 2.0) nu mai apar pe revolute.

PRISMATICELE raman placeholdere, etichetate NEVERIFICAT in xacro: documentul nu are
date de forta sau viteza pentru push rod-uri.

SEPARATIA, documentata in safety_limits.yaml si in SPEC_DERIVATE.md: URDF-ul poarta
CAPABILITATEA masinii, yaml-ul pragul TERAPEUTIC (mult mai mic, supravegheat la
runtime). Nu se sincronizeaza si nu se confunda.

colcon test: 8 teste, 0 erori, 0 esecuri.

File: rehab_exo_description/urdf/rehab_exo.urdf.xacro (robot description, xacro)
@@ -56,4 +56,17 @@
   <xacro:property name="gle_lo"  value="${glezna_min_deg * d2r}"/>
   <xacro:property name="gle_hi"  value="${glezna_max_deg * d2r}"/>
+  <!-- EFORT si VITEZA: DERIVATE din documentatie, nu alese. Formula si sursele in
+       urdf/SPEC_DERIVATE.md, generat din scripts/spec_derivate.py.
+         viteza = (rpm / 60) * 2*pi / raport_total
+         efort  = min(cuplu_motor * raport * eta, cuplu_nominal_reductor)
+       Cifrele vechi (120 Nm peste tot, 2.0 rad/s peste tot) nu aveau nicio sursa.
+       ACESTEA sunt CAPABILITATEA masinii; pragul terapeutic e in
+       config/safety_limits.yaml si e deliberat mult mai mic. -->
+  <xacro:property name="ef_sold"     value="176.7"/>
+  <xacro:property name="ef_genunchi" value="141.4"/>
+  <xacro:property name="ef_glezna"   value="52.0"/>
+  <xacro:property name="vi_sold"     value="1.5786"/>
+  <xacro:property name="vi_genunchi" value="1.9732"/>
+  <xacro:property name="vi_glezna"   value="1.5708"/>
   <xacro:arg name="controllers"
              default="$(find rehab_exo_description)/config/controllers.yaml"/>
@@ -111,5 +124,5 @@
     <origin xyz="0 0 0.485" rpy="0 0 0"/>
     <axis xyz="0 0 1"/>
-    <limit lower="0.0" upper="0.15" effort="500.0" velocity="0.05"/>
+    <limit lower="0.0" upper="0.15" effort="500.0" velocity="0.05"/><!-- NEVERIFICAT: coloana de ridicare, fara date in document -->
     <dynamics damping="50.0" friction="5.0"/>
   </joint>
@@ -259,5 +272,5 @@
     <origin xyz="0.160 ${sy * 0.260} 0.035" rpy="0 ${pi/2} 0"/>
     <axis xyz="0 -1 0"/>
-    <limit lower="${sold_lo}" upper="${sold_hi}" effort="120.0" velocity="2.0"/>
+    <limit lower="${sold_lo}" upper="${sold_hi}" effort="${ef_sold}" velocity="${vi_sold}"/>
     <dynamics damping="2.0" friction="1.0"/>
   </joint>
@@ -292,5 +305,5 @@
     <origin xyz="0.400 0 0" rpy="0 0 0"/>
     <axis xyz="1 0 0"/>
-    <limit lower="0.0" upper="0.08" effort="300.0" velocity="0.03"/>
+    <limit lower="0.0" upper="0.08" effort="300.0" velocity="0.03"/><!-- NEVERIFICAT: push rod fara date de forta sau viteza in document -->
     <dynamics damping="30.0" friction="3.0"/>
   </joint>
@@ -320,5 +333,5 @@
     <origin xyz="0 0 0" rpy="0 ${-pi/2} 0"/>
     <axis xyz="0 1 0"/>
-    <limit lower="${gen_lo}" upper="${gen_hi}" effort="120.0" velocity="2.0"/>
+    <limit lower="${gen_lo}" upper="${gen_hi}" effort="${ef_genunchi}" velocity="${vi_genunchi}"/>
     <dynamics damping="2.0" friction="1.0"/>
   </joint>
@@ -348,5 +361,5 @@
     <origin xyz="0 0 -0.400" rpy="0 0 0"/>
     <axis xyz="0 0 -1"/>
-    <limit lower="0.0" upper="0.08" effort="300.0" velocity="0.03"/>
+    <limit lower="0.0" upper="0.08" effort="300.0" velocity="0.03"/><!-- NEVERIFICAT: push rod fara date de forta sau viteza in document -->
     <dynamics damping="30.0" friction="3.0"/>
   </joint>
@@ -371,5 +384,5 @@
     <origin xyz="0 0 0" rpy="0 0 0"/>
     <axis xyz="0 -1 0"/>
-    <limit lower="${gle_lo}" upper="${gle_hi}" effort="120.0" velocity="2.0"/>
+    <limit lower="${gle_lo}" upper="${gle_hi}" effort="${ef_glezna}" velocity="${vi_glezna}"/>
     <dynamics damping="2.0" friction="1.0"/>
   </joint>

Commit message: fix(rehab): turatia gleznei -- cifra inventata inlocuita cu bobinaj parametrizat
Corectie ceruta la acceptarea M2, si e o incalcare a propriei reguli anti-fabricare.
Prima versiune folosea 1500 rpm pentru TBM(S)-6025. Cifra NU e in
SPEC_LLR_twin_din_PDF.md, care da pentru TBM doar cuplu continuu/varf, tensiuni, poli,
masa si inertie. Am ALES-O. Eticheta 'ipoteza' era corecta, provenienta lipsea -- iar o
ipoteza tot are nevoie de un DE UNDE. Istoricul ramane scris in cod, nu sters.

Turatia devine PARAMETRU pe bobinaj, cum cerea si specificatia modulului:
  A, 48 V -> 2900 rpm   (implicit: driverul e ADP-090-40 la 90 V [PDF Tabel 3.2 p.11])
  B, 24 V -> 2450 rpm
Ambele comunicate de autor pe 21 aug 2026 din foaia TBM-6025; NU sunt in extractul SPEC
de care dispun, deci raman marcate NEconfirmate la sursa.

CONSECINTA, exact cat se prevedea: viteza gleznei trece de la 1.5708 la 3.0369 rad/s --
aproape dublu. Efortul nu se schimba (acolo limiteaza reductorul), si exista o asertie
care cere sa nu se schimbe.

COMPLETITUDINEA analizei de prag, adaugata ca verificare: glezna e SINGURA articulatie
cu prag de randament in intervalul fizic (0,1).
  sold      eta* = 345/(0.9*245.45)  = 1.5617  -> peste 1, motorul limiteaza mereu
  genunchi  eta* = 178/(0.9*196.36)  = 1.0072  -> peste 1, dar la 0.7% de basculare
  glezna    eta* = 52/(0.706*100)    = 0.7365  -> singurul prag fizic
Deci analiza de prag e pusa unde conteaza, si acum se si DOVEDESTE ca acolo conteaza.
Genunchiul la 0.7% de basculare e o marja mai mica decat pare si merita masurata.

Selftest spec_derivate: 33 verificari (de la 27). colcon test: 8 teste verzi.

File: rehab_exo_description/urdf/rehab_exo.urdf.xacro (robot description, xacro)
@@ -68,5 +68,5 @@
   <xacro:property name="vi_sold"     value="1.5786"/>
   <xacro:property name="vi_genunchi" value="1.9732"/>
-  <xacro:property name="vi_glezna"   value="1.5708"/>
+  <xacro:property name="vi_glezna"   value="3.0369"/>
   <xacro:arg name="controllers"
              default="$(find rehab_exo_description)/config/controllers.yaml"/>

Commit message: update24sept2026

File: rehab_exo_description/urdf/rehab_exo.urdf.xacro (robot description, xacro)
@@ -184,4 +184,11 @@
   <material name="pants"><color rgba="0.25 0.25 0.28 1.0"/></material>
   <material name="shoe"><color rgba="0.10 0.10 0.10 1.0"/></material>
+  <!-- Culorile de instrumentatie fac lizibile componentele documentate. Geometria
+       lor este SCHEMATICA (fara cote in PDF), exclusiv visual: nu schimba masa,
+       coliziunile sau dinamica. -->
+  <material name="sensor_cuplu"><color rgba="0.95 0.55 0.05 1.0"/></material>
+  <material name="sensor_unghi"><color rgba="0.58 0.25 0.75 1.0"/></material>
+  <material name="sensor_forta"><color rgba="0.90 0.12 0.12 1.0"/></material>
+  <material name="sensor_rigla"><color rgba="0.10 0.75 0.70 1.0"/></material>
   <link name="world"/>
   <joint name="world_to_base" type="fixed">
@@ -340,7 +347,21 @@
       <inertia ixx="1.029333" ixy="0" ixz="0" iyy="0.874667" iyz="0" izz="0.461867"/>
     </inertial>
-    <visual>
-      <origin xyz="-0.1000 0.0000 0.2800" rpy="0 0 0"/>
-      <geometry><box size="0.2400 0.3400 0.5200"/></geometry>
+    <!-- Pacientul ramane o anvelopa antropometrica VIZUALA, nu un model biomecanic.
+         Volumele rotunjite de mai jos inlocuiesc paralelipipedul unic si sunt legate
+         vizual la bazin, umeri si coate. Coliziunea si inertialul raman neschimbate,
+         deci aceasta imbunatatire estetica NU schimba matematica simularii. -->
+    <visual>
+      <origin xyz="-0.1000 0.0000 0.0800" rpy="0 0 0"/>
+      <geometry><cylinder radius="0.1350" length="0.1600"/></geometry>
+      <material name="pants"/>
+    </visual>
+    <visual>
+      <origin xyz="-0.1000 0.0000 0.2450" rpy="0 0 0"/>
+      <geometry><cylinder radius="0.1300" length="0.2500"/></geometry>
+      <material name="cloth"/>
+    </visual>
+    <visual>
+      <origin xyz="-0.1000 0.0000 0.4200" rpy="0 0 0"/>
+      <geometry><cylinder radius="0.1650" length="0.1800"/></geometry>
       <material name="cloth"/>
     </visual>
@@ -366,4 +387,14 @@
     </visual>
     <visual>
+      <origin xyz="-0.1000 0.1700 0.4550" rpy="0 0 0"/>
+      <geometry><sphere radius="0.0650"/></geometry>
+      <material name="cloth"/>
+    </visual>
+    <visual>
+      <origin xyz="-0.1000 -0.1700 0.4550" rpy="0 0 0"/>
+      <geometry><sphere radius="0.0650"/></geometry>
+      <material name="cloth"/>
+    </visual>
+    <visual>
       <origin xyz="0.1300 0.2350 0.2350" rpy="0 1.5708 0"/>
       <geometry><cylinder radius="0.0400" length="0.2400"/></geometry>
@@ -373,4 +404,14 @@
       <origin xyz="0.1300 -0.2350 0.2350" rpy="0 1.5708 0"/>
       <geometry><cylinder radius="0.0400" length="0.2400"/></geometry>
+      <material name="skin"/>
+    </visual>
+    <visual>
+      <origin xyz="0.0000 0.2300 0.2450" rpy="0 0 0"/>
+      <geometry><sphere radius="0.0470"/></geometry>
+      <material name="skin"/>
+    </visual>
+    <visual>
+      <origin xyz="0.0000 -0.2300 0.2450" rpy="0 0 0"/>
+      <geometry><sphere radius="0.0470"/></geometry>
       <material name="skin"/>
     </visual>
@@ -421,4 +462,11 @@
     </visual>
     <visual>
+      <!-- M2210B la sold, intre iesirea reductorului si axul de transmisie.
+           Pozitia functionala vine din PDF; diametrul/grosimea sunt SCHEMATICE. -->
+      <origin xyz="0.0000 ${sy * 0.1175} 0.0000" rpy="1.5708 0 0"/>
+      <geometry><cylinder radius="0.0550" length="0.0250"/></geometry>
+      <material name="sensor_cuplu"/>
+    </visual>
+    <visual>
       <origin xyz="${g_coapsa_nom/2} 0.0000 0.0000" rpy="0 0 0"/>
       <geometry><box size="${g_coapsa_nom} 0.0500 0.0700"/></geometry>
@@ -459,4 +507,10 @@
       <geometry><cylinder radius="${g_d_genunchi/2}" length="0.0800"/></geometry>
       <material name="frame_gri"/>
+    </visual>
+    <visual>
+      <!-- M2210B la genunchi; doar reper vizual, fara coliziune/inertie. -->
+      <origin xyz="0.0000 ${sy * 0.0925} 0.0000" rpy="1.5708 0 0"/>
+      <geometry><cylinder radius="0.0470" length="0.0250"/></geometry>
+      <material name="sensor_cuplu"/>
     </visual>
     <collision>
@@ -486,4 +540,11 @@
     </visual>
     <visual>
+      <!-- Rigla electronica 406, montata longitudinal pe reglajul gambei.
+           Sectiunea este conventionala; canalul sau ramane explicit sintetic. -->
+      <origin xyz="${g_gamba_nom/2} ${sy * 0.0550} 0.0450" rpy="0 0 0"/>
+      <geometry><box size="${g_gamba_nom - 0.08} 0.0180 0.0180"/></geometry>
+      <material name="sensor_rigla"/>
+    </visual>
+    <visual>
       <origin xyz="${g_gamba_nom/2} ${sy * -0.1150} 0.0000" rpy="0 1.5708 0"/>
       <geometry><cylinder radius="0.0580" length="${g_gamba_nom - 0.05}"/></geometry>
@@ -537,4 +598,19 @@
       <geometry><box size="0.0250 0.1300 ${g_talpa_lungime}"/></geometry>
       <material name="frame_gri"/>
+    </visual>
+    <visual>
+      <!-- BWK216: senzorul dedicat de unghi al gleznei. Forma si cota de montaj
+           sunt schematice; prezenta si rolul sunt documentate in PDF. -->
+      <origin xyz="0.0000 ${sy * 0.0525} 0.0000" rpy="1.5708 0 0"/>
+      <geometry><cylinder radius="0.0280" length="0.0250"/></geometry>
+      <material name="sensor_unghi"/>
+    </visual>
+    <visual>
+      <!-- TR69-1500 sub talpa: forta Ff, apasare FN si moment MC. Blocul rosu
+           este numai un reper functional, nu model CAD si nu contact Gazebo. -->
+      <origin xyz="${g_glezna_offset - 0.018} ${sy * -0.0575} ${g_talpa_lungime/4}"
+              rpy="0 0 0"/>
+      <geometry><box size="0.0120 0.1050 0.1150"/></geometry>
+      <material name="sensor_forta"/>
     </visual>
     <visual>
